File: eagle/psas_c3.brd (EAGLE design)
At the start: 100 x 80 mm, 77 parts, among them IC1 CP2102, U1 MIC5219 3.3V, Y1 32MHz

Commit message: Added a few more recommended things to the schematic
Parts:
- removed C9: 100nF, Vibrogait_prototype:.0603-B-NOSILK
- removed Y1: 32MHz, Lilypad_Arduino_USB_v12:SPARKFUN-FREQCTRL_RESONATOR-SMD
- added C22, C26: 11pF, Vibrogait_prototype:.0603-B-NOSILK
- added C27, C28: 100nF, Vibrogait_prototype:.0603-B-NOSILK
- added Q1: 32 MHz, crystal:FC-12M
- added R6: 0, rcl_custom:.0603-B-NOSILK
Connections:
- removed net N$11: U$1.46, Y1.1
- net 3.3V: no longer C9.1, U$1.1
- net GND: now also C26.2, C27.2, C28.2; no longer C9.2, Y1.2
- net N$12: now also Q1.2; no longer U$1.47, Y1.3
- net PTD5: no longer IC1.23
- net PTD6: no longer IC1.24
