File: eagle/psas_c3.brd (EAGLE design)
At the start: 100 x 80 mm, 81 parts, among them IC1 CP2102, Q1 32 MHz, U1 MIC5219 3.3V

Commit message: Fixed alignment issues on schematic
Connections:
- removed net N$24: C1.1
- removed net N$26: LED1.2, U2.P$18, U2.P$19, U2.P$2, U2.P$3, U2.P$9
- new net N$11: R6.2, U$1.47
- net GND: now also C22.2
- net N$12: now also C22.1, R6.1
- net N$15: now also C26.1, Q1.1, U$1.46; no longer C21.1, R1.1, S2.A2
- net RESET: now also C21.1, R1.1, S2.A2
- net VBUS: now also C1.1, LED1.2, U2.P$18, U2.P$19, U2.P$2, U2.P$3, U2.P$9
Changed lines of the file:
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@@
 <contactref element="U$1" pad="3"/>
 <contactref element="C8" pad="2"/>
+<contactref element="C22" pad="2"/>
 <wire x1="-87.05" y1="-160.02" x2="-87.05" y2="-165.1" width="0" layer="19" extent="1-1"/>
 <wire x1="-87.05" y1="-170.18" x2="-87.05" y2="-165.1" width="0" layer="19" extent="1-1"/>
@@
 <wire x1="-82.385" y1="-320.33" x2="-82.55" y2="-209.55" width="0" layer="19" extent="1-1"/>
 <wire x1="-89.37" y1="-327.66" x2="-82.385" y2="-320.33" width="0" layer="19" extent="1-1"/>
-<wire x1="-89.37" y1="-347.98" x2="-89.37" y2="-327.66" width="0" layer="19" extent="1-1"/>
+<wire x1="-89.37" y1="-342.9" x2="-89.37" y2="-327.66" width="0" layer="19" extent="1-1"/>
+<wire x1="-89.37" y1="-347.98" x2="-89.37" y2="-342.9" width="0" layer="19" extent="1-1"/>
 <wire x1="-89.37" y1="-353.06" x2="-89.37" y2="-347.98" width="0" layer="19" extent="1-1"/>
 <wire x1="-89.37" y1="-358.14" x2="-89.37" y2="-353.06" width="0" layer="19" extent="1-1"/>
@@
 <contactref element="TP5" pad="1"/>
 <contactref element="IC1" pad="8"/>
-<wire x1="-56.68" y1="-29.21" x2="-60.96" y2="-66.04" width="0" layer="19" extent="1-1"/>
+<contactref element="LED1" pad="2"/>
+<contactref element="U2" pad="P$9"/>
+<contactref element="C1" pad="1"/>
+<contactref element="U2" pad="P$3"/>
+<contactref element="U2" pad="P$18"/>
+<contactref element="U2" pad="P$2"/>
+<contactref element="U2" pad="P$19"/>
+<wire x1="-56.68" y1="-58.97" x2="-60.96" y2="-66.04" width="0" layer="19" extent="1-1"/>
+<wire x1="-56.68" y1="-29.21" x2="-56.68" y2="-58.97" width="0" layer="19" extent="1-1"/>
 <wire x1="-56.11" y1="-22.62" x2="-56.68" y2="-29.21" width="0" layer="19" extent="1-1"/>
 <wire x1="-56.91" y1="-21.82" x2="-56.11" y2="-22.62" width="0" layer="19" extent="1-1"/>
 <wire x1="-35.59" y1="22.995" x2="-56.91" y2="-21.82" width="0" layer="19" extent="1-1"/>
+<wire x1="-17.205" y1="30.48" x2="-35.59" y2="22.995" width="0" layer="19" extent="1-1"/>
+<wire x1="-17.205" y1="30.98" x2="-17.205" y2="30.48" width="0" layer="19" extent="1-1"/>
+<wire x1="-15.74" y1="32.445" x2="-17.205" y2="30.98" width="0" layer="19" extent="1-1"/>
+<wire x1="-15.24" y1="32.445" x2="-15.74" y2="32.445" width="0" layer="19" extent="1-1"/>
+<wire x1="-14.74" y1="28.515" x2="-17.205" y2="30.48" width="0" layer="19" extent="1-1"/>
+<wire x1="-30.01" y1="46.99" x2="-15.74" y2="32.445" width="0" layer="19" extent="1-1"/>
 </signal>
 <signal name="V+">
@@
 <wire x1="-25.88" y1="19.135" x2="-78.74" y2="-313.69" width="0" layer="19" extent="1-1"/>
 </signal>
-<signal name="N$15">
-<contactref element="R1" pad="1"/>
-<contactref element="S2" pad="A2"/>
-<contactref element="C21" pad="1"/>
-<wire x1="-82.385" y1="-324.83" x2="-90.97" y2="-327.66" width="0" layer="19" extent="1-1"/>
-<wire x1="-90.97" y1="-317.5" x2="-90.97" y2="-327.66" width="0" layer="19" extent="1-1"/>
-</signal>
 <signal name="RESET">
 <contactref element="U$1" pad="33"/>
 <contactref element="JTAG1" pad="10"/>
+<contactref element="R1" pad="1"/>
+<contactref element="C21" pad="1"/>
+<contactref element="S2" pad="A2"/>
+<wire x1="-82.385" y1="-324.83" x2="-90.97" y2="-327.66" width="0" layer="19" extent="1-1"/>
+<wire x1="-90.97" y1="-317.5" x2="-90.97" y2="-327.66" width="0" layer="19" extent="1-1"/>
+<wire x1="-74.93" y1="-207.01" x2="-90.97" y2="-317.5" width="0" layer="19" extent="1-1"/>
 <wire x1="-20.405" y1="24.11" x2="-74.93" y2="-207.01" width="0" layer="19" extent="1-1"/>
 </signal>
-<signal name="N$26">
-<contactref element="U2" pad="P$2"/>
-<contactref element="U2" pad="P$9"/>
-<contactref element="U2" pad="P$3"/>
-<contactref element="U2" pad="P$19"/>
-<contactref element="LED1" pad="2"/>
-<contactref element="U2" pad="P$18"/>
-<wire x1="-14.74" y1="28.515" x2="-56.68" y2="-58.97" width="0" layer="19" extent="1-1"/>
-<wire x1="-17.205" y1="30.48" x2="-14.74" y2="28.515" width="0" layer="19" extent="1-1"/>
-<wire x1="-17.205" y1="30.98" x2="-17.205" y2="30.48" width="0" layer="19" extent="1-1"/>
-<wire x1="-15.74" y1="32.445" x2="-17.205" y2="30.98" width="0" layer="19" extent="1-1"/>
-<wire x1="-15.24" y1="32.445" x2="-15.74" y2="32.445" width="0" layer="19" extent="1-1"/>
-</signal>
-<signal name="N$24">
-<contactref element="C1" pad="1"/>
+<signal name="N$11">
+<contactref element="U$1" pad="47"/>
+<contactref element="R6" pad="2"/>
+<wire x1="-22.88" y1="19.135" x2="-89.37" y2="-337.82" width="0" layer="19" extent="1-1"/>
 </signal>
 <signal name="N$12">
+<contactref element="R6" pad="1"/>
+<contactref element="C22" pad="1"/>
 <contactref element="Q1" pad="2"/>
+<wire x1="-90.97" y1="-337.82" x2="-90.97" y2="-342.9" width="0" layer="19" extent="1-1"/>
+<wire x1="-89.32" y1="-332.74" x2="-90.97" y2="-337.82" width="0" layer="19" extent="1-1"/>
+</signal>
+<signal name="N$15">
+<contactref element="U$1" pad="46"/>
+<contactref element="C26" pad="1"/>
+<contactref element="Q1" pad="1"/>
+<wire x1="-91.02" y1="-332.74" x2="-90.97" y2="-347.98" width="0" layer="19" extent="1-1"/>
+<wire x1="-22.38" y1="19.135" x2="-91.02" y2="-332.74" width="0" layer="19" extent="1-1"/>
 </signal>
 </signals>

Commit message: Fixed alignment issues on schematic
Connections:
- new net N$23: U$1.48
- net PTB1: no longer U$1.48
Changed lines of the file:
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@@
 <contactref element="U$1" pad="18"/>
 <contactref element="JP17" pad="2"/>
-<contactref element="U$1" pad="48"/>
-<wire x1="-23.38" y1="19.135" x2="-86.36" y2="-293.37" width="0" layer="19" extent="1-1"/>
-<wire x1="-25.88" y1="26.585" x2="-23.38" y2="19.135" width="0" layer="19" extent="1-1"/>
+<wire x1="-25.88" y1="26.585" x2="-86.36" y2="-293.37" width="0" layer="19" extent="1-1"/>
 </signal>
 <signal name="PTB0">
@@
 <wire x1="-22.38" y1="19.135" x2="-91.02" y2="-332.74" width="0" layer="19" extent="1-1"/>
 </signal>
+<signal name="N$23">
+<contactref element="U$1" pad="48"/>
+</signal>
 </signals>

Commit message: made fixes to schematic
Connections:
- new net N$24: IC1.24
- new net VREFH: C27.1, U$1.1
- net 3.3V: now also C28.1
- net N$23: now also IC1.23; no longer U$1.48
- net PTA2: now also IC1.25
- net PTB1: now also U$1.48; no longer JP17.2
Changed lines of the file:
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@@
 <contactref element="JTAG1" pad="1"/>
 <contactref element="R1" pad="2"/>
+<contactref element="C28" pad="1"/>
+<wire x1="-89.37" y1="-317.5" x2="-90.97" y2="-358.14" width="0" layer="19" extent="1-1"/>
 <wire x1="-85.09" y1="-209.55" x2="-89.37" y2="-317.5" width="0" layer="19" extent="1-1"/>
 <wire x1="-90.97" y1="-184.15" x2="-85.09" y2="-209.55" width="0" layer="19" extent="1-1"/>
@@
 <contactref element="U$1" pad="13"/>
 <contactref element="JP4" pad="3"/>
-<wire x1="-27.855" y1="25.61" x2="-83.82" y2="-222.25" width="0" layer="19" extent="1-1"/>
+<contactref element="IC1" pad="25"/>
+<wire x1="-27.855" y1="25.61" x2="-54.61" y2="-18.02" width="0" layer="19" extent="1-1"/>
+<wire x1="-83.82" y1="-222.25" x2="-54.61" y2="-18.02" width="0" layer="19" extent="1-1"/>
 </signal>
 <signal name="N$30">
@@
 <signal name="PTB1">
 <contactref element="U$1" pad="18"/>
-<contactref element="JP17" pad="2"/>
-<wire x1="-25.88" y1="26.585" x2="-86.36" y2="-293.37" width="0" layer="19" extent="1-1"/>
+<contactref element="U$1" pad="48"/>
+<wire x1="-25.88" y1="26.585" x2="-23.38" y2="19.135" width="0" layer="19" extent="1-1"/>
 </signal>
 <signal name="PTB0">
@@
 <wire x1="-22.38" y1="19.135" x2="-91.02" y2="-332.74" width="0" layer="19" extent="1-1"/>
 </signal>
+<signal name="VREFH">
+<contactref element="U$1" pad="1"/>
+<contactref element="C27" pad="1"/>
+<wire x1="-27.855" y1="19.61" x2="-90.97" y2="-353.06" width="0" layer="19" extent="1-1"/>
+</signal>
 <signal name="N$23">
-<contactref element="U$1" pad="48"/>
+<contactref element="IC1" pad="23"/>
+</signal>
+<signal name="N$24">
+<contactref element="IC1" pad="24"/>
 </signal>
 </signals>

Commit message: rev2 of schematic
Parts:
- removed JP10, JP16, JP18, JP19, JP20, JP9: (no value), SparkFun-v5:1X03
- removed JP11: (no value), SparkFun-v5:1X04
- removed JP12, JP17, JP7: (no value), SparkFun-v5:1X02
- removed JP13, JP14: M01PTH, SparkFun-v5:1X01
- removed JP15: (no value), SparkFun-v5:1X05
- removed JP21: (no value), SparkFun-v5:1X06
- JP3, JP8: device SparkFun-v5:1X02 -> pinhead:2X02
- JP4: device SparkFun-v5:1X03 -> pinhead:2X04
- JP5: device SparkFun-v5:1X03 -> pinhead:2X03
- JP6: device SparkFun-v5:1X03 -> pinhead:2X05
- moved JP4 143.7 mm to (-95.2, -365.8)
- moved JP6 141.7 mm to (-102.9, -373.4)
- moved JP3 137.4 mm to (-97.8, -354.3)
- moved JP5 136.9 mm to (-105.4, -363.2)
- moved JP8 133.1 mm to (-124.5, -370.8)
Connections:
- net N$11 renamed XTA
- net N$15 renamed XTB
- net N$16 renamed RFIO
- net N$20 renamed VR_PA
- net RESET renamed PTA20/!RESET
- removed net N$13: JP21.5, U$1.53
- removed net N$23: IC1.23
- removed net N$24 (its old number): IC1.24
- removed net N$5: JP21.3, U$1.51
- removed net N$7: JP21.4, U$1.52
- removed net PTA19: JP6.3, U$1.16
- removed net PTA4: JP19.3, U$1.12
- new net DIO2: JP8.2, U$1.51
- new net DIO3: JP8.1, U$1.52
- new net DIO4: JP8.3, U$1.53
- new net PTE30: JP6.3, U$1.9
- net 3.3V: now also LED1.2; no longer RP2.1
- net D+: now also D3.CATHODE; no longer D1.CATHODE
- net DIO5/CLKOUT: now also JP8.4; no longer JP21.6
- net PTA1: now also IC1.26; no longer JP3.2
- net PTA18: now also JP2.1; no longer JP5.3
- net PTA2: no longer JP4.3
- net PTA3: no longer JP20.3
- net PTB0: now also JP3.1, U$1.48; no longer JP18.3
- net PTB1: now also JP3.2; no longer U$1.48
- net PTB17: now also JP3.3; no longer JP15.1, JP4.1
- net PTB2: now also JP3.4; no longer JP18.2
- net PTC1: now also JP4.2; no longer JP20.1
- net PTC2: now also JP4.4; no longer JP19.1
- net PTC3: now also JP4.6; no longer JP5.2
- net PTC4: now also JP4.8; no longer JP6.2, JP9.3
- net PTC5: now also JP4.7; no longer JP12.2
- net PTC6: now also JP4.5; no longer JP10.3, JP11.3
- net PTC7: now also JP4.3; no longer JP11.4
- net PTD0: now also JP5.2; no longer JP9.2
- net PTD4: now also JP5.4; no longer JP13.1, JP7.2
- net PTD5: now also JP5.6; no longer JP8.2
- net PTD6: now also JP5.5; no longer JP15.5, JP3.1
- net PTD7: now also JP5.3; no longer JP11.1, JP15.4, JP4.2
- net PTE0: now also JP6.2; no longer JP16.2, JP19.2, JP6.1
- net PTE1: now also JP6.4; no longer JP15.3, JP16.1, JP20.2, JP5.1
- net PTE16: now also JP6.10; no longer JP8.1, JP9.1
- net PTE17: now also JP6.9; no longer JP12.1, JP7.1
- net PTE18: now also JP6.7; no longer JP10.2, JP17.1
- net PTE19: now also JP6.5; no longer JP10.1, JP11.2, JP18.1
- net PTE2: now also JP6.6; no longer JP14.1
- net PTE3: now also JP6.8; no longer JP15.2, JP16.3
- net VBUS: now also D1.CATHODE, RP2.1; no longer LED1.2

Commit message: took care of ERC
Parts:
- removed C28: 100nF, Vibrogait_prototype:.0603-B-NOSILK
- added C9: 100nF, Vibrogait_prototype:.0603-B-NOSILK
- ANT1: value (none) -> Antenna
- CF1: value (none) -> CF1
- R3, R4, R5: value (none) -> 1k
- RT1: value (none) -> 10K (NTC)
- U2: value (none) -> MCP73871
Connections:
- removed net VREFH: C27.1, U$1.1
- net 3.3V: now also C27.1, C9.1, U$1.1; no longer C28.1
- net GND: now also C9.2, IC1.23; no longer C28.2
Changed lines of the file:
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@@
 </autorouter>
 <elements>
-<element name="ANT1" library="discrete" package="PAD-01" value="" x="-31.75" y="29.21"/>
+<element name="ANT1" library="discrete" package="PAD-01" value="Antenna" x="-31.75" y="29.21"/>
 <element name="C1" library="rcl_custom" package=".0603-B-NOSILK" value="10uF" x="-29.21" y="46.99"/>
 <element name="C10" library="rcl_custom" package=".0603-B-NOSILK" value="10p" x="-16.51" y="41.91"/>
@@
 <attribute name="MFG" value="Murata Electronics North America" x="-41.91" y="36.83" size="1.778" layer="27" display="off"/>
 </element>
-<element name="CF1" library="Vibrogait_prototype" package="USB-MICRO-B-PTH-HIROSE" value="" x="-34.29" y="20.32"/>
+<element name="CF1" library="Vibrogait_prototype" package="USB-MICRO-B-PTH-HIROSE" value="CF1" x="-34.29" y="20.32"/>
 <element name="JP1" library="Vibrogait_prototype" package="SPARKFUN-CONNECTORS_JST-2-SMD-VERT" value="battery_connector" x="-38.1" y="6.35"/>
 <element name="JP2" library="SparkFun-v5" package="1X02" value="" x="-38.1" y="29.21"/>
@@
 <element name="RP1" library="rcl_custom" package=".0603-B-NOSILK" value="5k" x="-36.83" y="46.99"/>
 <element name="RP3" library="rcl_custom" package=".0603-B-NOSILK" value="100k" x="-33.02" y="46.99"/>
-<element name="RT1" library="Vibrogait_prototype" package="R1206" value="" x="-45.72" y="45.72"/>
+<element name="RT1" library="Vibrogait_prototype" package="R1206" value="10K (NTC)" x="-45.72" y="45.72"/>
 <element name="S1" library="Vibrogait_prototype" package="SWITCH-SPDT" value="" x="-15.24" y="6.35"/>
 <element name="TP1" library="microbuilder" package="1X01_ROUND" value="" x="-46.99" y="29.21">
@@
 <attribute name="PROD_ID" value="VREG-09872" x="-43.18" y="29.21" size="1.778" layer="27" display="off"/>
 </element>
-<element name="U2" library="microbuilder" package="QFN20_4MM" value="" x="-15.24" y="30.48"/>
+<element name="U2" library="microbuilder" package="QFN20_4MM" value="MCP73871" x="-15.24" y="30.48"/>
 <element name="R2" library="rcl_custom" package=".0603-A-NOSILK" value="0" x="-45.72" y="-24.13"/>
 <element name="IC1" library="silabs" package="MLP28" value="CP2102" x="-54.61" y="-20.32">
@@
 <element name="R14" library="rcl_custom" package=".0603-B-NOSILK" value="1M" x="-55.88" y="-54.61"/>
 <element name="LED1" library="Vibrogait_prototype" package="KINGBRITE_RGBLED_1.6X1.26" value="" x="-55.88" y="-58.42"/>
-<element name="R3" library="rcl_custom" package=".0603-B-NOSILK" value="" x="-55.88" y="-62.23"/>
-<element name="R4" library="rcl_custom" package=".0603-B-NOSILK" value="" x="-55.88" y="-66.04"/>
-<element name="R5" library="rcl_custom" package=".0603-B-NOSILK" value="" x="-55.88" y="-69.85"/>
+<element name="R3" library="rcl_custom" package=".0603-B-NOSILK" value="1k" x="-55.88" y="-62.23"/>
+<element name="R4" library="rcl_custom" package=".0603-B-NOSILK" value="1k" x="-55.88" y="-66.04"/>
+<element name="R5" library="rcl_custom" package=".0603-B-NOSILK" value="1k" x="-55.88" y="-69.85"/>
 <element name="TP5" library="microbuilder" package="1X01_ROUND" value="" x="-60.96" y="-66.04">
 <attribute name="BOM" value="EXCLUDE" x="-60.96" y="-66.04" size="1.778" layer="27" display="off"/>
@@
 <attribute name="MFG" value="Murata Electronics North America" x="-90.17" y="-353.06" size="1.778" layer="27" display="off"/>
 </element>
-<element name="C28" library="Vibrogait_prototype" package=".0603-B-NOSILK" value="100nF" x="-90.17" y="-358.14">
-<attribute name="MPN" value="GRM188R71C104KA01D" x="-90.17" y="-358.14" size="1.778" layer="27" display="off"/>
-<attribute name="DPN" value="490-1532-1-ND" x="-90.17" y="-358.14" size="1.778" layer="27" display="off"/>
-<attribute name="DIST" value="Digi-Key" x="-90.17" y="-358.14" size="1.778" layer="27" display="off"/>
-<attribute name="MFG" value="Murata Electronics North America" x="-90.17" y="-358.14" size="1.778" layer="27" display="off"/>
-</element>
 <element name="JP3" library="pinhead" package="2X02" value="" x="-97.79" y="-354.33"/>
 <element name="JP4" library="pinhead" package="2X04" value="" x="-95.25" y="-365.76"/>
@@
 <element name="JP6" library="pinhead" package="2X05" value="" x="-102.87" y="-373.38"/>
 <element name="JP8" library="pinhead" package="2X02" value="" x="-124.46" y="-370.84"/>
+<element name="C9" library="Vibrogait_prototype" package=".0603-B-NOSILK" value="100nF" x="-125.73" y="-378.46">
+<attribute name="MPN" value="GRM188R71C104KA01D" x="-125.73" y="-378.46" size="1.778" layer="27" display="off"/>
+<attribute name="DPN" value="490-1532-1-ND" x="-125.73" y="-378.46" size="1.778" layer="27" display="off"/>
+<attribute name="MFG" value="Murata Electronics North America" x="-125.73" y="-378.46" size="1.778" layer="27" display="off"/>
+<attribute name="DIST" value="Digi-Key" x="-125.73" y="-378.46" size="1.778" layer="27" display="off"/>
+</element>
 </elements>
 <signals>
@@
 <contactref element="C21" pad="2"/>
 <contactref element="C26" pad="2"/>
-<contactref element="U$1" pad="2"/>
-<contactref element="C27" pad="2"/>
-<contactref element="C28" pad="2"/>
-<contactref element="U$1" pad="3"/>
 <contactref element="C8" pad="2"/>
 <contactref element="C22" pad="2"/>
@@
 <contactref element="U2" pad="P$17"/>
 <contactref element="C1" pad="2"/>
+<contactref element="C27" pad="2"/>
+<contactref element="C9" pad="2"/>
+<contactref element="U$1" pad="3"/>
+<contactref element="U$1" pad="2"/>
+<contactref element="IC1" pad="23"/>
 <wire x1="-87.05" y1="-160.02" x2="-87.05" y2="-165.1" width="0" layer="19" extent="1-1"/>
 <wire x1="-87.05" y1="-170.18" x2="-87.05" y2="-165.1" width="0" layer="19" extent="1-1"/>
@@
 <wire x1="-56.91" y1="-19.82" x2="-54.61" y2="-20.32" width="0" layer="19" extent="1-1"/>
 <wire x1="-56.7125" y1="-18.2175" x2="-56.91" y2="-19.82" width="0" layer="19" extent="1-1"/>
+<wire x1="-53.61" y1="-18.02" x2="-54.61" y2="-20.32" width="0" layer="19" extent="1-1"/>
 <wire x1="-46.62" y1="-24.13" x2="-54.61" y2="-20.32" width="0" layer="19" extent="1-1"/>
 <wire x1="-44.82" y1="-24.13" x2="-46.62" y2="-24.13" width="0" layer="19" extent="1-1"/>
-<wire x1="-37.1" y1="4.35" x2="-44.82" y2="-24.13" width="0" layer="19" extent="1-1"/>
+<wire x1="-37.1" y1="4.35" x2="-53.61" y2="-18.02" width="0" layer="19" extent="1-1"/>
 <wire x1="-27.855" y1="20.11" x2="-37.1" y2="4.35" width="0" layer="19" extent="1-1"/>
 <wire x1="-27.855" y1="20.61" x2="-27.855" y2="20.11" width="0" layer="19" extent="1-1"/>
@@
 <wire x1="-89.37" y1="-347.98" x2="-89.37" y2="-342.9" width="0" layer="19" extent="1-1"/>
 <wire x1="-89.37" y1="-353.06" x2="-89.37" y2="-347.98" width="0" layer="19" extent="1-1"/>
-<wire x1="-89.37" y1="-358.14" x2="-89.37" y2="-353.06" width="0" layer="19" extent="1-1"/>
+<wire x1="-124.93" y1="-378.46" x2="-89.37" y2="-353.06" width="0" layer="19" extent="1-1"/>
 </signal>
 <signal name="VOUT">
@@
 <contactref element="U$1" pad="55"/>
 <contactref element="C8" pad="1"/>
-<contactref element="U$1" pad="56"/>
 <contactref element="U$1" pad="43"/>
 <contactref element="U$1" pad="35"/>
@@
 <contactref element="JTAG1" pad="1"/>
 <contactref element="R1" pad="2"/>
-<contactref element="C28" pad="1"/>
 <contactref element="LED1" pad="2"/>
-<wire x1="-89.37" y1="-317.5" x2="-90.97" y2="-358.14" width="0" layer="19" extent="1-1"/>
+<contactref element="C9" pad="1"/>
+<contactref element="C27" pad="1"/>
+<contactref element="U$1" pad="1"/>
+<contactref element="U$1" pad="56"/>
+<wire x1="-90.97" y1="-353.06" x2="-126.53" y2="-378.46" width="0" layer="19" extent="1-1"/>
+<wire x1="-89.37" y1="-317.5" x2="-90.97" y2="-353.06" width="0" layer="19" extent="1-1"/>
 <wire x1="-85.09" y1="-209.55" x2="-89.37" y2="-317.5" width="0" layer="19" extent="1-1"/>
 <wire x1="-90.97" y1="-184.15" x2="-85.09" y2="-209.55" width="0" layer="19" extent="1-1"/>
@@
 <wire x1="-27.38" y1="19.135" x2="-56.68" y2="-58.97" width="0" layer="19" extent="1-1"/>
 <wire x1="-26.88" y1="19.135" x2="-27.38" y2="19.135" width="0" layer="19" extent="1-1"/>
+<wire x1="-27.855" y1="19.61" x2="-27.38" y2="19.135" width="0" layer="19" extent="1-1"/>
 <wire x1="-20.88" y1="19.135" x2="-26.88" y2="19.135" width="0" layer="19" extent="1-1"/>
 <wire x1="-20.405" y1="23.11" x2="-20.88" y2="19.135" width="0" layer="19" extent="1-1"/>
@@
 <wire x1="-22.38" y1="19.135" x2="-91.02" y2="-332.74" width="0" layer="19" extent="1-1"/>
 </signal>
-<signal name="VREFH">
-<contactref element="U$1" pad="1"/>
-<contactref element="C27" pad="1"/>
-<wire x1="-27.855" y1="19.61" x2="-90.97" y2="-353.06" width="0" layer="19" extent="1-1"/>
-</signal>
 <signal name="N$24">

Commit message: two out of three revisions done
Parts:
- removed ANT1: Antenna, discrete:PAD-01
- added U$2: SMAJ716-ND, SMAJ16-ND:SMAJ716-ND
Connections:
- net N$19: now also U$2.P$3; no longer ANT1.1
Changed lines of the file:
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@@
 <?xml version="1.0" encoding="utf-8"?>
 <!DOCTYPE eagle SYSTEM "eagle.dtd">
-<eagle version="7.3.0">
+<eagle version="7.4.0">
 <drawing>
 <settings>
@@
 </autorouter>
 <elements>
-<element name="ANT1" library="discrete" package="PAD-01" value="Antenna" x="-31.75" y="29.21"/>
 <element name="C1" library="rcl_custom" package=".0603-B-NOSILK" value="10uF" x="-29.21" y="46.99"/>
 <element name="C10" library="rcl_custom" package=".0603-B-NOSILK" value="10p" x="-16.51" y="41.91"/>
@@
 <attribute name="DIST" value="Digi-Key" x="-125.73" y="-378.46" size="1.778" layer="27" display="off"/>
 </element>
+<element name="U$2" library="SMAJ16-ND" package="SMAJ716-ND" value="SMAJ716-ND" x="-121.92" y="-383.54"/>
 </elements>
 <signals>
@@
 <contactref element="C8" pad="1"/>
 <contactref element="U$1" pad="43"/>
-<contactref element="U$1" pad="35"/>
-<contactref element="C18" pad="1"/>
 <contactref element="JTAG1" pad="1"/>
 <contactref element="R1" pad="2"/>
@@
 <contactref element="U$1" pad="1"/>
 <contactref element="U$1" pad="56"/>
+<contactref element="C18" pad="1"/>
+<contactref element="U$1" pad="35"/>
 <wire x1="-90.97" y1="-353.06" x2="-126.53" y2="-378.46" width="0" layer="19" extent="1-1"/>
 <wire x1="-89.37" y1="-317.5" x2="-90.97" y2="-353.06" width="0" layer="19" extent="1-1"/>
@@
 <signal name="N$19">
 <contactref element="C15" pad="2"/>
-<contactref element="ANT1" pad="1"/>
-<wire x1="-41.11" y1="41.91" x2="-31.75" y2="29.21" width="0" layer="19" extent="1-1"/>
+<contactref element="U$2" pad="P$3"/>
+<wire x1="-41.11" y1="41.91" x2="-121.92" y2="-383.032" width="0" layer="19" extent="1-1"/>
 </signal>
 <signal name="VR_PA">
