File: eagle/psas_c3.brd (EAGLE design)
At the start: 100 x 80 mm, 78 parts, among them IC1 CP2102, Q1 32 MHz, U1 MIC5219 3.3V, U2 MCP73871

Commit message: Revert "revisions"
This reverts commit 38aaf88b81013dcc018781bf82979bc3fff6647d, reversing
changes made to 2f30e97817f685fc14312947979bc5bd385c959f.
Parts:
- JP3: device pinhead:2X04 -> pinhead:2X02
- JP4: device pinhead:2X07 -> pinhead:2X04
- JP5: device pinhead:2X05 -> pinhead:2X03
- JP6: device pinhead:2X09 -> pinhead:2X05
- moved JP3 90.5 mm to (-97.8, -354.3)
- moved JP5 86.5 mm to (-105.4, -363.2)
- moved JP6 82.9 mm to (-102.9, -373.4)
- moved JP4 80.2 mm to (-95.2, -365.8)
- moved JP7 21.6 mm to (-175.3, -389.9)
Connections:
- removed net RESET(RF): JP7.2, U$1.48
- new net N$25: JP3.1
- net PTB0: now also U$1.48; no longer JP3.1, JP3.2, JP7.1
- net PTB1: now also JP3.2; no longer JP3.3, JP3.4
- net PTB17: now also JP3.3; no longer JP3.7, JP3.8
- net PTB2: now also JP3.4; no longer JP3.5, JP3.6
- net PTC1: no longer JP4.1
- net PTC2: no longer JP4.3
- net PTC3: no longer JP4.5
- net PTC4: no longer JP4.7
- net PTC5: now also JP4.7; no longer JP4.10, JP4.9
- net PTC6: now also JP4.5; no longer JP4.11, JP4.12
- net PTC7: now also JP4.3; no longer JP4.14
- net PTD0: no longer JP5.1
- net PTD4: no longer JP5.3
- net PTD5: no longer JP5.5
- net PTD6: now also JP5.5; no longer JP5.7, JP5.8
- net PTD7: now also JP5.3; no longer JP5.10, JP5.9
- net PTE0: no longer JP6.1
- net PTE1: no longer JP6.3
- net PTE16: no longer JP6.9
- net PTE17: now also JP6.9; no longer JP6.11, JP6.12
- net PTE18: now also JP6.7; no longer JP6.13, JP6.14
- net PTE19: now also JP6.5; no longer JP6.15, JP6.16
- net PTE2: no longer JP6.5
- net PTE3: no longer JP6.7
- net PTE30: now also JP6.3; no longer JP6.17, JP6.18

Commit message: added bypass cap for vdd2, pin header for RESET(RF), double row pin header for each port on MCU, added pullup on RX/TX with jpin header for jumper, added pin header for battery status, 1000mAh battery, added pin header for transceiver GPIO, took away 0 ohm resistor on ground for MCU, added bypass caps to VBAT1 and VBAT2, made test points 20/1000 in, grouped stuff on board to help jake with initial layout
Parts:
- removed D2, D3: (no value), Vibrogait_prototype:SOD-123
- removed R2: 0, rcl_custom:.0603-A-NOSILK
- removed TP12, TP13, TP14: (no value), microbuilder:1X01_ROUND
- added C28, C29: 100nF, Vibrogait_prototype:.0603-B-NOSILK
- added JP10: (no value), pinhead:2X08
- added JP11: (no value), pinhead:2X02
- added JP9: (no value), pinhead:2X03
- added R420, R69: 4.7k, rcl_custom:.0603-B-NOSILK
- JP3: device pinhead:2X02 -> pinhead:1X02
- JP4: device pinhead:2X04 -> pinhead:2X07
- JP5: device pinhead:2X03 -> pinhead:2X05
- JP6: device pinhead:2X05 -> pinhead:2X09
- JP7: device pinhead:1X02 -> pinhead:2X04
- JP8: device pinhead:2X02 -> pinhead:2X04
- TP1, TP10, TP11, TP15, TP2, TP3, TP4, TP5, TP6, TP7, TP8, TP9: device microbuilder:1X01_ROUND -> microbuilder:TESTPOINT_ROUND_0.5MM
- moved C9 445.8 mm to (45.7, 33.0)
- moved C27 412.3 mm to (54.6, 33.0)
- moved C21 397.8 mm to (74.9, 34.3)
- moved C26 397.8 mm to (74.9, 14.0)
- moved C22 397.8 mm to (74.9, 19.1)
- moved Q1 397.8 mm to (74.9, 29.2)
- moved R1 397.8 mm to (74.9, 44.5)
- moved R6 397.8 mm to (74.9, 24.1)
- moved S2 397.8 mm to (78.7, 39.4)
- moved U1 122.1 mm to (73.7, 64.8), turned to 270 degrees
- moved S1 118.8 mm to (88.9, 63.5)
- moved JP1 118.1 mm to (57.1, 76.2)
- moved IC1 116.8 mm to (29.2, 61.0), turned to 180 degrees
- moved C8 87.6 mm to (45.7, 36.8)
- moved JP3 85.2 mm to (-175.3, -389.9)
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- renumbered RP2 to R411
Connections:
- removed net DIO2: JP8.2, U$1.51
- removed net DIO3: JP8.1, U$1.52
- removed net DIO4: JP8.3, U$1.53
- new net N$26: JP10.10, JP10.9, U$1.12
- new net N$27: JP10.13, JP10.14, U$1.16
- new net N$28: JP11.1, R69.1
- new net N$29: JP11.3, R420.1
- new net RESET(RF): JP3.2, U$1.48
- net !PG: now also JP9.1, JP9.2
- net 3.3V: now also C28.1, C29.1, JP11.2, JP11.4, TP3.P$1; no longer TP3.1
- net D+: no longer D3.CATHODE
- net D-: no longer D2.CATHODE
- net DIO5/CLKOUT: now also JP8.7, JP8.8; no longer JP8.4
- net GND: now also C28.2, C29.2, TP4.P$1; no longer D2.ANODE, D3.ANODE, IC1.23, R2.1, R2.2, TP4.1, TP9.1
- net N$11: now also TP8.P$1; no longer TP8.1
- net N$13: now also TP10.P$1; no longer TP10.1
- net N$15: now also TP11.P$1; no longer TP11.1
- net N$16: now also JP8.1, JP8.2, U$1.51; no longer JTAG1.6, TP12.1
- net N$20: now also JP8.3, JP8.4, U$1.52; no longer JTAG1.8, TP13.1
- net N$23: now also JP8.5, JP8.6, U$1.53; no longer JTAG1.7, TP14.1
- net N$25: now also IC1.23, TP9.P$1; no longer JP3.1
- net N$5: now also TP6.P$1; no longer TP6.1
- net N$7: now also TP7.P$1; no longer TP7.1
- net PTA0: now also JP10.1, JP10.2
- net PTA1: now also JP10.3, JP10.4, R69.2
- net PTA18: now also JP10.11, JP10.12
- net PTA2: now also JP10.5, JP10.6, R420.2
- net PTA20/!RESET: now also JP10.15, JP10.16
- net PTA3: now also JP10.7, JP10.8
- net PTB0: now also JP3.1, JP7.1, JP7.2; no longer U$1.48
- net PTB1: now also JP7.3, JP7.4; no longer JP3.2
- net PTB17: now also JP7.7, JP7.8; no longer JP3.3
- net PTB2: now also JP7.5, JP7.6; no longer JP3.4
- net PTC1: now also JP4.1
- net PTC2: now also JP4.3
- net PTC3: now also JP4.5
- net PTC4: now also JP4.7
- net PTC5: now also JP4.10, JP4.9; no longer JP4.7
- net PTC6: now also JP4.11, JP4.12; no longer JP4.5
- net PTC7: now also JP4.13, JP4.14; no longer JP4.3
- net PTD0: now also JP5.1
- net PTD4: now also JP5.3
- net PTD5: now also JP5.5
- net PTD6: now also JP5.7, JP5.8; no longer JP5.5
- net PTD7: now also JP5.10, JP5.9; no longer JP5.3
- net PTE1: now also JP6.3
- net PTE16: now also JP6.9
- net PTE17: now also JP6.11, JP6.12; no longer JP6.9
- net PTE18: now also JP6.13, JP6.14; no longer JP6.7
- net PTE19: now also JP6.15, JP6.16; no longer JP6.5
- net PTE2: now also JP6.5
- net PTE3: now also JP6.7
- net PTE30: now also JP6.17, JP6.18; no longer JP6.3
- net STAT1/LBO: now also JP9.5, JP9.6
- net STAT2: now also JP9.3, JP9.4
- net V+: now also TP1.P$1; no longer TP1.1
- net VBUS: now also TP5.P$1; no longer TP5.1
- net VOUT: now also TP2.P$1; no longer TP2.1
- net VR_PA: now also TP15.P$1; no longer TP15.1

Commit message: Board layout update and DRC for OSH
Parts:
- moved JP5 547.5 mm to (94.3, 65.9), turned to 90 degrees
- moved JP4 545.5 mm to (88.1, 76.0)
- moved JP10 530.1 mm to (3.45, 52.9), turned to 90 degrees
- moved JP11 525.2 mm to (15.1, 30.0)
- moved R69 520.7 mm to (13.9, 25.1), turned to 180 degrees
- moved JP9 515.1 mm to (26.1, 36.5)
- moved R420 512.9 mm to (14.0, 21.7), turned to 180 degrees
- moved JP8 505.8 mm to (52.9, 24.7), turned to 180 degrees
- moved JP7 500.2 mm to (9.63, 68.3)
- moved TP15 498.0 mm to (83.7, 43.6)
- moved JP6 485.6 mm to (54.1, 12.3), turned to 180 degrees
- moved TP7 484.8 mm to (33.9, 73.1)
- moved JP3 483.7 mm to (40.3, 43.1), turned to 270 degrees
- moved TP6 482.6 mm to (32.5, 73.1)
- moved U$2 478.3 mm to (96.5, 41.9), turned to 270 degrees
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Connections:
- net PTA2: no longer IC1.25

Commit message: board update
Parts:
- moved C25 48.4 mm to (85.8, 36.5), turned to 270 degrees
- moved JTAG1 46.4 mm to (58.8, 47.1), turned to 270 degrees
- moved R420 43.6 mm to (57.0, 28.8), turned to 270 degrees
- moved JP11 40.7 mm to (55.7, 33.2)
- moved JP10 37.9 mm to (38.0, 37.3)
- moved R69 37.6 mm to (50.9, 31.9)
- moved JP6 36.1 mm to (87.5, 26.2), turned to 0 degrees
- moved JP2 30.4 mm to (48.5, 46.6), turned to 270 degrees
- moved JP7 28.7 mm to (36.5, 58.0)
- moved C6 27.7 mm to (73.7, 54.2)
- moved C5 27.3 mm to (73.7, 52.3)
- moved LED1 26.4 mm to (49.0, 56.5)
- moved C8 26.3 mm to (67.1, 34.7), turned to 180 degrees
- moved JP9 25.3 mm to (45.9, 52.3), turned to 180 degrees
- moved C29 25.1 mm to (67.1, 40.5)
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Routing:
- net 3.3V: track 0.00 -> 27.4 mm
- net DIO5/CLKOUT: track 0.00 -> 20.7 mm
- net N$23: track 0.00 -> 18.9 mm
- net N$16: track 0.00 -> 17.3 mm
- net N$20: track 0.00 -> 17.3 mm
- net PTA1: track 0.00 -> 14.2 mm
- net VR_PA: track 0.00 -> 11.9 mm
- net RFIO: track 0.00 -> 11.7 mm
- net N$14: track 0.00 -> 11.3 mm
- net N$7: track 0.00 -> 8.06 mm
- net N$17: track 0.00 -> 6.27 mm
- net N$22: track 0.00 -> 6.05 mm
- net PTB0: track 0.00 -> 5.99 mm
- net N$5: track 0.00 -> 5.94 mm
- net N$21: track 0.00 -> 5.03 mm
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
Commit message: board update
Parts:
- moved JP3 5.02 mm to (37.6, 51.2)
- moved JP5 4.79 mm to (90.2, 67.6), turned to 0 degrees
- moved C27 3.62 mm to (69.7, 39.8)
- moved C29 3.62 mm to (69.6, 37.9)
- moved C8 3.62 mm to (69.6, 32.0)
- moved C9 3.62 mm to (69.6, 33.9)
- moved C28 3.62 mm to (69.6, 35.8)
- moved JP10 3.48 mm to (41.5, 37.3)
- moved TP1 3.23 mm to (66.3, 63.7)
- moved JP7 2.21 mm to (36.3, 60.2), turned to 90 degrees
- moved C22 1.39 mm to (74.9, 35.2)
- moved C23 1.39 mm to (80.4, 37.7)
- moved Q1 1.39 mm to (75.9, 37.7)
- moved C26 1.39 mm to (77.8, 37.7)
- moved R6 1.39 mm to (74.1, 37.7)
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Routing:
- net 3.3V: track 27.4 -> 74.4 mm
- net PTA1: track 14.2 -> 55.1 mm
- net PTA2: track 2.54 -> 30.4 mm
- net PTD7: track 2.54 -> 29.2 mm
- net PTD6: track 2.54 -> 27.1 mm
- net PTD5: track 2.54 -> 25.5 mm
- net VBUS: track 0.00 -> 18.7 mm
- net VOUT: track 0.00 -> 17.8 mm
- net V+: track 0.00 -> 12.9 mm
- net PTA3: track 2.54 -> 13.7 mm
- net PTA0: track 2.54 -> 12.8 mm
- net N$30: track 0.00 -> 10.2 mm
- net PTA18: track 2.54 -> 12.0 mm
- net STAT1/LBO: track 0.00 -> 7.33 mm
- net N$8: track 0.00 -> 5.65 mm
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
Commit message: Board changes
Parts:
- moved JP6 43.2 mm to (43.8, 23.7), turned to 90 degrees
- moved C2 41.2 mm to (24.7, 66.7)
- moved C19 41.2 mm to (9.92, 68.1)
- moved C20 41.2 mm to (15.1, 75.9)
- moved C24 41.2 mm to (11.8, 68.2)
- moved C7 41.2 mm to (24.2, 74.2)
- moved D1 41.2 mm to (5.97, 71.1)
- moved IC1 41.2 mm to (6.31, 65.9)
- moved R14 41.2 mm to (16.9, 75.9)
- moved R411 41.2 mm to (15.2, 64.2)
- moved S1 41.2 mm to (33.2, 71.1)
- moved TP2 41.2 mm to (23.8, 65.2)
- moved TP5 41.2 mm to (12.2, 65.7)
- moved TP6 41.2 mm to (1.18, 69.5)
- moved TP7 41.2 mm to (1.18, 71.1)
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Routing:
- net PTA1: track 55.1 -> 0.00 mm
- net PTE16: track 0.00 -> 41.1 mm
- net PTE17: track 0.00 -> 39.0 mm
- net PTE18: track 0.00 -> 37.0 mm
- net PTE19: track 0.00 -> 34.9 mm
- net PTE30: track 0.00 -> 32.9 mm
- net PTA2: track 30.4 -> 0.00 mm
- net PTD4: track 0.00 -> 28.8 mm
- net N$27: track 2.54 -> 25.4 mm
- net N$26: track 2.54 -> 20.8 mm
- net PTA0: track 12.8 -> 29.1 mm
- net 3.3V: track 74.4 -> 59.2 mm
- net V+: track 12.9 -> 0.50 mm
- net PTA18: track 12.0 -> 22.3 mm
- net VR_PA: track 11.9 -> 21.2 mm
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
Commit message: Board update
Parts:
- moved C21 58.8 mm to (8.58, 14.9)
- moved C4 55.7 mm to (10.7, 71.7)
- moved TP4 52.4 mm to (14.1, 28.5)
- moved R1 49.5 mm to (34.1, 24.3)
- moved JP1 40.9 mm to (14.6, 75.9), turned to 0 degrees
- moved C6 40.6 mm to (25.9, 52.9), turned to 270 degrees
- moved C5 36.1 mm to (29.0, 52.9), turned to 270 degrees
- moved RP1 36.0 mm to (29.8, 74.8), turned to 0 degrees
- moved TP3 34.8 mm to (29.0, 56.8)
- moved RP3 34.5 mm to (29.8, 76.8), turned to 0 degrees
- moved TP6 30.8 mm to (2.68, 38.7)
- moved TP7 30.6 mm to (2.63, 40.5)
- moved D1 26.1 mm to (3.30, 45.1), turned to 270 degrees
- moved RT1 24.3 mm to (41.1, 75.8), turned to 0 degrees
- moved TP9 22.2 mm to (15.7, 42.7)
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Routing:
- net 3.3V: track 59.2 -> 162.6 mm, vias 0 -> 6
- net VBUS: track 18.7 -> 102.7 mm, vias 0 -> 5
- net PTA1: track 0.00 -> 72.7 mm, vias 0 -> 3
- net PTE2: track 0.00 -> 63.7 mm, vias 0 -> 2
- net DIO5/CLKOUT: track 27.6 -> 71.3 mm, vias 0 -> 2
- net PTE3: track 0.00 -> 40.5 mm, vias 0 -> 2
- net STAT1/LBO: track 0.00 -> 39.3 mm
- net PTA0: track 29.1 -> 66.4 mm
- net V+: track 0.50 -> 34.6 mm
- net PTC3: track 2.54 -> 35.9 mm
- net PTC2: track 2.54 -> 35.2 mm
- net PTC1: track 2.54 -> 34.5 mm
- net RESET(RF): track 0.00 -> 31.3 mm, vias 0 -> 1
- net PTA2: track 0.00 -> 30.7 mm, vias 0 -> 1
- net STAT2: track 0.00 -> 28.6 mm
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
Commit message: Board update
Parts:
- moved TP15 3.76 mm to (87.9, 37.6)
Routing:
- net PTE0: track 0.00 -> 85.3 mm, vias 0 -> 2
- net PTE1: track 2.54 -> 79.5 mm, vias 0 -> 2
- net 3.3V: track 162.6 -> 211.7 mm
- net PTC6: track 2.54 -> 42.1 mm, vias 0 -> 1
- net PTC7: track 2.54 -> 42.1 mm, vias 0 -> 1
- net PTC5: track 2.54 -> 38.0 mm, vias 0 -> 1
- net PTD0: track 2.54 -> 34.9 mm, vias 0 -> 1
- net PTC4: track 2.54 -> 34.9 mm, vias 0 -> 1
- net N$27: track 2.54 -> 27.9 mm
- net PTA18: track 11.1 -> 33.4 mm
