File: eagle/psas_c3.sch (EAGLE design)
At the start: 81 parts, among them IC1 CP2102, Q1 32 MHz, U1 MIC5219 3.3V

Commit message: made fixes to schematic
Connections:
- new net N$24: IC1.RTS
- new net VREFH: C27.1, U$1.VREFH
- net 3.3V: now also C28.1
- net N$23: now also IC1.CTS; no longer U$1.RESET(RF)
- net PTA2: now also IC1.RXD
- net PTB1: now also U$1.RESET(RF); no longer JP17.2
Changed lines of the file:
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@@
 <setting verticaltext="up"/>
 </settings>
-<grid distance="0.1" unitdist="inch" unit="inch" style="dots" multiple="1" display="yes" altdistance="0.01" altunitdist="inch" altunit="inch"/>
+<grid distance="0.1" unitdist="inch" unit="inch" style="lines" multiple="1" display="yes" altdistance="0.01" altunitdist="inch" altunit="inch"/>
 <layers>
 <layer number="1" name="Top" color="4" fill="1" visible="no" active="no"/>
@@
 <attribute name="VALUE" x="62.484" y="337.439" size="1.778" layer="96" rot="MR180"/>
 </instance>
-<instance part="P+5" gate="G$1" x="124.333" y="315.087" rot="R180"/>
-<instance part="RP2" gate="R" x="124.333" y="325.247" rot="R90"/>
+<instance part="P+5" gate="G$1" x="124.46" y="314.96" rot="R180"/>
+<instance part="RP2" gate="R" x="124.46" y="325.12" rot="R90"/>
 <instance part="C20" gate="CE" x="43.18" y="363.22" rot="MR180"/>
 <instance part="R14" gate="R" x="38.1" y="365.76" smashed="yes" rot="R90">
@@
 <pinref part="U$1" gate="G$1" pin="VDDA"/>
 <wire x1="185.42" y1="259.08" x2="185.42" y2="274.32" width="0.1524" layer="91"/>
+<pinref part="C28" gate="CE" pin="1"/>
 <wire x1="185.42" y1="274.32" x2="185.42" y2="279.4" width="0.1524" layer="91"/>
 <wire x1="177.8" y1="271.78" x2="177.8" y2="274.32" width="0.1524" layer="91"/>
@@
 <pinref part="P+5" gate="G$1" pin="3.3V"/>
 <pinref part="RP2" gate="R" pin="1"/>
-<wire x1="124.333" y1="315.087" x2="124.333" y2="320.167" width="0.1524" layer="91"/>
+<wire x1="124.46" y1="314.96" x2="124.46" y2="320.04" width="0.1524" layer="91"/>
 </segment>
 <segment>
@@
 <pinref part="U$1" gate="G$1" pin="PTA1"/>
 <wire x1="226.06" y1="187.96" x2="307.34" y2="187.96" width="0.1524" layer="91"/>
-<wire x1="307.34" y1="187.96" x2="426.72" y2="187.96" width="0.1524" layer="91"/>
 <label x="359.1814" y="189.7888" size="1.778" layer="95" rot="R180"/>
 <wire x1="307.34" y1="144.78" x2="307.34" y2="187.96" width="0.1524" layer="91"/>
-<junction x="307.34" y="187.96"/>
 <pinref part="JP3" gate="G$1" pin="2"/>
 <wire x1="330.2" y1="144.78" x2="307.34" y2="144.78" width="0.1524" layer="91"/>
 <label x="266.7" y="187.96" size="1.778" layer="95"/>
 <label x="314.96" y="144.78" size="1.778" layer="95"/>
-</segment>
-<segment>
-<wire x1="119.3292" y1="353.2124" x2="135.9154" y2="353.2124" width="0.1524" layer="91"/>
-<wire x1="135.9154" y1="353.2124" x2="135.9154" y2="297.0784" width="0.1524" layer="91"/>
-<wire x1="135.9154" y1="297.0784" x2="238.76" y2="297.0784" width="0.1524" layer="91"/>
-<wire x1="238.76" y1="297.0784" x2="238.76" y2="281.813" width="0.1524" layer="91"/>
-<wire x1="238.76" y1="281.813" x2="429.3362" y2="281.813" width="0.1524" layer="91"/>
-<wire x1="429.3362" y1="281.813" x2="429.3362" y2="187.96" width="0.1524" layer="91"/>
-<wire x1="429.3362" y1="187.96" x2="426.72" y2="187.96" width="0.1524" layer="91"/>
+<wire x1="307.34" y1="187.96" x2="429.26" y2="187.96" width="0.1524" layer="91"/>
+<wire x1="429.26" y1="187.96" x2="429.26" y2="281.94" width="0.1524" layer="91"/>
+<junction x="307.34" y="187.96"/>
+<wire x1="429.26" y1="281.94" x2="238.76" y2="281.94" width="0.1524" layer="91"/>
+<wire x1="238.76" y1="281.94" x2="238.76" y2="297.18" width="0.1524" layer="91"/>
+<wire x1="119.38" y1="353.06" x2="137.16" y2="353.06" width="0.1524" layer="91"/>
+<wire x1="137.16" y1="353.06" x2="137.16" y2="297.18" width="0.1524" layer="91"/>
+<wire x1="238.76" y1="297.18" x2="137.16" y2="297.18" width="0.1524" layer="91"/>
 </segment>
 </net>
@@
 <pinref part="U$1" gate="G$1" pin="PTA2"/>
 <wire x1="226.06" y1="185.42" x2="304.8" y2="185.42" width="0.1524" layer="91"/>
-<wire x1="304.8" y1="185.42" x2="431.7746" y2="185.3946" width="0.1524" layer="91"/>
 <label x="359.156" y="187.2742" size="1.778" layer="95" rot="R180"/>
 <wire x1="304.8" y1="132.08" x2="304.8" y2="185.42" width="0.1524" layer="91"/>
-<junction x="304.8" y="185.42"/>
 <pinref part="JP4" gate="G$1" pin="3"/>
 <wire x1="330.2" y1="132.08" x2="304.8" y2="132.08" width="0.1524" layer="91"/>
@@
 </segment>
 <segment>
-<wire x1="119.2022" y1="355.727" x2="138.4808" y2="355.7016" width="0.1524" layer="91"/>
-<wire x1="138.4808" y1="355.7016" x2="138.4554" y2="299.72" width="0.1524" layer="91"/>
-<wire x1="138.4554" y1="299.72" x2="241.3" y2="299.72" width="0.1524" layer="91"/>
+<wire x1="139.7" y1="355.6" x2="139.7" y2="299.72" width="0.1524" layer="91"/>
+<wire x1="139.7" y1="299.72" x2="241.3" y2="299.72" width="0.1524" layer="91"/>
 <wire x1="241.3" y1="299.72" x2="241.3" y2="284.48" width="0.1524" layer="91"/>
 <wire x1="241.3" y1="284.48" x2="431.8" y2="284.48" width="0.1524" layer="91"/>
 <wire x1="431.8" y1="284.48" x2="431.8" y2="185.42" width="0.1524" layer="91"/>
+<pinref part="IC1" gate="G$1" pin="RXD"/>
+<wire x1="119.38" y1="355.6" x2="139.7" y2="355.6" width="0.1524" layer="91"/>
 </segment>
 </net>
@@
 <pinref part="RP2" gate="R" pin="2"/>
 <pinref part="IC1" gate="G$1" pin="!RST"/>
-<wire x1="124.333" y1="330.327" x2="119.38" y2="330.2" width="0.1524" layer="91"/>
+<wire x1="124.46" y1="330.2" x2="119.38" y2="330.2" width="0.1524" layer="91"/>
 <pinref part="IC1" gate="G$1" pin="DCD"/>
-<wire x1="119.38" y1="345.44" x2="124.333" y2="345.567" width="0.1524" layer="91"/>
-<wire x1="124.333" y1="345.567" x2="124.333" y2="343.027" width="0.1524" layer="91"/>
-<junction x="124.333" y="330.327"/>
+<wire x1="119.38" y1="345.44" x2="124.46" y2="345.44" width="0.1524" layer="91"/>
+<wire x1="124.46" y1="345.44" x2="124.46" y2="342.9" width="0.1524" layer="91"/>
+<junction x="124.46" y="330.2"/>
 <pinref part="IC1" gate="G$1" pin="DTR"/>
-<wire x1="124.333" y1="343.027" x2="124.333" y2="330.327" width="0.1524" layer="91"/>
-<wire x1="119.38" y1="347.98" x2="124.333" y2="348.107" width="0.1524" layer="91"/>
-<wire x1="124.333" y1="348.107" x2="124.333" y2="345.567" width="0.1524" layer="91"/>
-<junction x="124.333" y="345.567"/>
+<wire x1="124.46" y1="342.9" x2="124.46" y2="330.2" width="0.1524" layer="91"/>
+<wire x1="119.38" y1="347.98" x2="124.46" y2="347.98" width="0.1524" layer="91"/>
+<wire x1="124.46" y1="347.98" x2="124.46" y2="345.44" width="0.1524" layer="91"/>
+<junction x="124.46" y="345.44"/>
 <pinref part="IC1" gate="G$1" pin="DSR"/>
-<wire x1="119.38" y1="350.52" x2="124.333" y2="350.647" width="0.1524" layer="91"/>
-<wire x1="124.333" y1="350.647" x2="124.333" y2="348.107" width="0.1524" layer="91"/>
-<junction x="124.333" y="348.107"/>
+<wire x1="119.38" y1="350.52" x2="124.46" y2="350.52" width="0.1524" layer="91"/>
+<wire x1="124.46" y1="350.52" x2="124.46" y2="347.98" width="0.1524" layer="91"/>
+<junction x="124.46" y="347.98"/>
 <pinref part="IC1" gate="G$1" pin="RI"/>
-<wire x1="119.38" y1="342.9" x2="124.333" y2="343.027" width="0.1524" layer="91"/>
-<junction x="124.333" y="343.027"/>
+<wire x1="119.38" y1="342.9" x2="124.46" y2="342.9" width="0.1524" layer="91"/>
+<junction x="124.46" y="342.9"/>
 </segment>
 </net>
@@
 <label x="266.7" y="177.8" size="1.778" layer="95"/>
 <label x="375.92" y="142.24" size="1.778" layer="95"/>
+<wire x1="365.76" y1="177.8" x2="365.76" y2="195.58" width="0.1524" layer="91"/>
+<wire x1="365.76" y1="195.58" x2="411.48" y2="195.58" width="0.1524" layer="91"/>
+<junction x="365.76" y="177.8"/>
 </segment>
 </net>
@@
 <pinref part="U$1" gate="G$1" pin="PTB1"/>
 <wire x1="185.42" y1="238.76" x2="160.02" y2="238.76" width="0.1524" layer="91"/>
-<wire x1="160.02" y1="238.76" x2="160.147" y2="287.02" width="0.1524" layer="91"/>
-<pinref part="JP17" gate="G$1" pin="2"/>
-<wire x1="160.147" y1="287.02" x2="43.434" y2="287.02" width="0.1524" layer="91"/>
+<wire x1="160.02" y1="238.76" x2="160.02" y2="287.02" width="0.1524" layer="91"/>
 <label x="160.02" y="256.54" size="1.778" layer="95" rot="R90"/>
+<pinref part="U$1" gate="G$1" pin="RESET(RF)"/>
+<wire x1="228.6" y1="261.62" x2="226.06" y2="261.62" width="0.1524" layer="91"/>
+<wire x1="228.6" y1="287.02" x2="228.6" y2="261.62" width="0.1524" layer="91"/>
+<wire x1="228.6" y1="287.02" x2="160.02" y2="287.02" width="0.1524" layer="91"/>
+<wire x1="43.18" y1="287.02" x2="160.02" y2="287.02" width="0.1524" layer="91"/>
+<junction x="160.02" y="287.02"/>
 </segment>
 </net>
@@
 </segment>
 </net>
-<net name="N$25" class="0">
-<segment>
-<wire x1="365.76" y1="177.8254" x2="365.8108" y2="196.3928" width="0.1524" layer="91"/>
-<wire x1="365.8108" y1="196.3928" x2="411.7594" y2="196.3928" width="0.1524" layer="91"/>
-</segment>
-</net>
 <net name="VREFH" class="0">
 <segment>
-<wire x1="185.4454" y1="251.46" x2="170.18" y2="251.46" width="0.1524" layer="91"/>
-<wire x1="170.18" y1="251.46" x2="170.18" y2="279.4" width="0.1524" layer="91"/>
-</segment>
-<segment>
+<wire x1="170.18" y1="251.46" x2="170.18" y2="274.32" width="0.1524" layer="91"/>
+<pinref part="U$1" gate="G$1" pin="VREFH"/>
+<wire x1="170.18" y1="274.32" x2="170.18" y2="279.4" width="0.1524" layer="91"/>
+<wire x1="185.42" y1="251.46" x2="170.18" y2="251.46" width="0.1524" layer="91"/>
+<pinref part="C27" gate="CE" pin="1"/>
 <wire x1="165.1" y1="271.78" x2="165.1" y2="274.32" width="0.1524" layer="91"/>
 <wire x1="165.1" y1="274.32" x2="170.18" y2="274.32" width="0.1524" layer="91"/>
+<junction x="170.18" y="274.32"/>
 </segment>
 </net>
@@
 <net name="N$23" class="0">
 <segment>
-<pinref part="U$1" gate="G$1" pin="RESET(RF)"/>
-<wire x1="228.6" y1="261.62" x2="226.06" y2="261.62" width="0.1524" layer="91"/>
-<wire x1="228.6" y1="287.02" x2="228.6" y2="261.62" width="0.1524" layer="91"/>
-</segment>
-</net>
+<pinref part="IC1" gate="G$1" pin="CTS"/>
+<wire x1="119.38" y1="360.68" x2="127" y2="360.68" width="0.1524" layer="91"/>
+</segment>
+</net>
+<net name="N$24" class="0">
+<segment>
+<pinref part="IC1" gate="G$1" pin="RTS"/>
+<wire x1="119.38" y1="358.14" x2="127" y2="358.14" width="0.1524" layer="91"/>
+</segment>
+</net>

Commit message: rev2 of schematic
Parts:
- removed JP10, JP16, JP18, JP19, JP20, JP9: (no value), SparkFun-v5:M03PTH
- removed JP11: (no value), SparkFun-v5:M04PTH
- removed JP12, JP17, JP7: (no value), SparkFun-v5:M02PTH
- removed JP13, JP14: M01PTH, SparkFun-v5:M01PTH
- removed JP15: (no value), SparkFun-v5:M05PTH
- removed JP21: (no value), SparkFun-v5:M06SIP
- JP3, JP8: device SparkFun-v5:M02PTH -> pinhead:PINHD-2X2
- JP4: device SparkFun-v5:M03PTH -> pinhead:PINHD-2X4
- JP5: device SparkFun-v5:M03PTH -> pinhead:PINHD-2X3
- JP6: device SparkFun-v5:M03PTH -> pinhead:PINHD-2X5
Connections:
- net N$11 renamed XTA
- net N$15 renamed XTB
- net N$16 renamed RFIO
- net N$20 renamed VR_PA
- net RESET renamed PTA20/!RESET
- removed net N$13: JP21.5, U$1.DIO4
- removed net N$23: IC1.CTS
- removed net N$24 (its old number): IC1.RTS
- removed net N$5: JP21.3, U$1.DIO2
- removed net N$7: JP21.4, U$1.DIO3
- removed net PTA19: JP6.3, U$1.PTA19/XTAL0
- removed net PTA4: JP19.3, U$1.PTA4
- new net DIO2: JP8.2, U$1.DIO2
- new net DIO3: JP8.1, U$1.DIO3
- new net DIO4: JP8.3, U$1.DIO4
- new net PTE30: JP6.3, U$1.PTE30
- net 3.3V: now also LED1.COMMON_ANODE; no longer RP2.1
- net D+: now also D3.CATHODE; no longer D1.CATHODE
- net DIO5/CLKOUT: now also JP8.4; no longer JP21.6
- net PTA1: now also IC1.TXD; no longer JP3.2
- net PTA18: now also JP2.1; no longer JP5.3
- net PTA2: no longer JP4.3
- net PTA3: no longer JP20.3
- net PTB0: now also JP3.1, U$1.RESET(RF); no longer JP18.3
- net PTB1: now also JP3.2; no longer U$1.RESET(RF)
- net PTB17: now also JP3.3; no longer JP15.1, JP4.1
- net PTB2: now also JP3.4; no longer JP18.2
- net PTC1: now also JP4.2; no longer JP20.1
- net PTC2: now also JP4.4; no longer JP19.1
- net PTC3: now also JP4.6; no longer JP5.2
- net PTC4: now also JP4.8; no longer JP6.2, JP9.3
- net PTC5: now also JP4.7; no longer JP12.2
- net PTC6: now also JP4.5; no longer JP10.3, JP11.3
- net PTC7: now also JP4.3; no longer JP11.4
- net PTD0: now also JP5.2; no longer JP9.2
- net PTD4: now also JP5.4; no longer JP13.1, JP7.2
- net PTD5: now also JP5.6; no longer JP8.2
- net PTD6: now also JP5.5; no longer JP15.5, JP3.1
- net PTD7: now also JP5.3; no longer JP11.1, JP15.4, JP4.2
- net PTE0: now also JP6.2; no longer JP16.2, JP19.2, JP6.1
- net PTE1: now also JP6.4; no longer JP15.3, JP16.1, JP20.2, JP5.1
- net PTE16: now also JP6.10; no longer JP8.1, JP9.1
- net PTE17: now also JP6.9; no longer JP12.1, JP7.1
- net PTE18: now also JP6.7; no longer JP10.2, JP17.1
- net PTE19: now also JP6.5; no longer JP10.1, JP11.2, JP18.1
- net PTE2: now also JP6.6; no longer JP14.1
- net PTE3: now also JP6.8; no longer JP15.2, JP16.3
- net VBUS: now also D1.CATHODE, RP2.1; no longer LED1.COMMON_ANODE
Other:
- note added: "3.7V 400mAh lipo cell battery"
- note added: "Clock selection When connected, MCU uses 32MHz for clock"
- note added: "PORTB"
- note added: "PORTC"
- note added: "PORTD"
- note added: "PORTE"
- note added: "RESET(RF) is suppose to be controlled by a GPIO according to the databook"
- note added: "This is for the transciever GPIO ..yes it has GPIO read the databook"
- note removed: "I2C0"
- note removed: "I2C0_SCL"
- note removed: "I2C0_SDA"
- note removed: "I2C1"
- note removed: "I2C1_SCL"
- note removed: "I2C1_SDA"
- note removed: "RX"
- note removed: "SPI0"
- note removed: "SPI0_MISO"
- note removed: "SPI0_MOSI"
- note removed: "SPI0_PCS0"
- note removed: "SPI0_SCK"
- note removed: "SPI1"
- note removed: "SPI1_MISO"
- note removed: "SPI1_MOSI"
- note removed: "SPI1_PCS0"
- note removed: "SPI1_SCK"
- note removed: "TX"
- note removed: "Transciever GPIO"
- note removed: "UART0"
- note removed: "UART1"
- note removed: "UART2"
- moved on the sheet: ANT1, C1, C10, C11, C12, C13, C14, C15, C16, C17, C19, C20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

Commit message: took care of ERC
Parts:
- removed C28: 100nF, Vibrogait_prototype:C-EU0603-B-NOSILK
- added C9: 100nF, Vibrogait_prototype:C-EU0603-B-NOSILK
- ANT1: value (none) -> Antenna
- CF1: value (none) -> CF1
- R3, R4, R5: value (none) -> 1k
- RT1: value (none) -> 10K (NTC)
- U2: value (none) -> MCP73871
Connections:
- removed net VREFH: C27.1, U$1.VREFH
- net 3.3V: now also C27.1, C9.1, U$1.VREFH; no longer C28.1
- net GND: now also C9.2, IC1.CTS; no longer C28.2
Other:
- note added: "bypass for VDDA"
- note added: "bypass for VREFH"
- moved on the sheet: ANT1, C1, C10, C11, C12, C13, C14, C15, C16, C17, C18, C19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

Commit message: two out of three revisions done
Parts:
- removed ANT1: Antenna, discrete:ANTENNA
- added U$2: SMAJ716-ND, SMAJ16-ND:SMAJ716-ND
Connections:
- net N$19: now also U$2.CENTERCONDUCTOR; no longer ANT1.1
Other:
- note added: "Antenna"
- note added: "SMA J716-ND"
- moved on the sheet: C18, C8, JP8
